File: sensor-node-ext/noise-amp/noise-amp.kicad_pcb (KiCad board)
At the start: 2 copper layers, 30.5 x 38.1 mm, 19 parts, among them J1 INSELECT, K1 XLR3, P1 MIC, P2 PIEZO, P3 PIEZO, P4 PIEZO, U1 MCP6002

Commit message: Sensor node ext designs
Routing:
- added copper zone on F.Cu, net GND
Changed lines of the file:
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@@
   (segment (start 168.91 89.408) (end 168.91 86.788) (width 0.25) (layer B.Cu) (net 2) (status 10))
   (segment (start 168.91 86.788) (end 167.212 85.09) (width 0.25) (layer B.Cu) (net 2) (status 20))
-  (segment (start 170.688 70.612) (end 170.688 70.104) (width 0.8) (layer B.Cu) (net 4) (status C00000))
-  (segment (start 170.688 70.104) (end 169.164 68.58) (width 0.8) (layer B.Cu) (net 4) (status 400000))
+  (segment (start 170.688 70.612) (end 170.688 70.104) (width 0.8) (layer B.Cu) (net 4))
+  (segment (start 170.688 70.104) (end 169.164 68.58) (width 0.8) (layer B.Cu) (net 4))
   (via (at 165.862 76.962) (size 0.9) (drill 0.7) (layers F.Cu B.Cu) (net 4))
   (segment (start 165.862 76.962) (end 165.862 70.358) (width 0.8) (layer F.Cu) (net 4))
@@
     (connect_pads (clearance 0.508))
     (min_thickness 0.254)
+    (fill yes (arc_segments 16) (thermal_gap 0.508) (thermal_bridge_width 0.508))
+    (polygon
+      (pts
+        (xy 162.56 60.96) (xy 163.83 59.69) (xy 191.77 59.69) (xy 193.04 60.96) (xy 193.04 96.52)
+        (xy 191.77 97.79) (xy 163.83 97.79) (xy 162.56 96.52)
+      )
+    )
+  )
+  (zone (net 3) (net_name GND) (layer F.Cu) (hatch edge 0.508)
+    (connect_pads (clearance 0.508))
+    (min_thickness 0.254)
