File: sensor-node-ext/sensor-block/sensor-node-ext.kicad_pcb (KiCad board)
At the start: 2 copper layers, 99.3 x 38.9 mm, 32 parts, among them J1 DB9, J2 DB9, J3 DB9, K1 XLR3, K2 XLR3, K3 XLR3, K4 XLR3, K5 XLR3, K6 XLR3, P1 XBEE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

Commit message: Sensor node ext designs
Parts:
- removed J2: DB9, Connect:DB9FC
- removed Q3, Q4, Q5: 2N7000, TO_SOT_Packages_THT:TO-92_Inline_Wide
- removed R4: 100k, Resistors_SMD:R_0805_HandSoldering
- added IMU1: IMU, w_pin_strip:pin_socket_9, F.Cu at (148.6, 69.3)
- Q1, Q2: value 2N7000 -> BS170
- R3: moved to B.Cu
- moved R3 12.6 mm to (71.8, 57.1), turned to 0 degrees
- moved K6 10.4 mm to (68.1, 70.2), turned to 90 degrees
- moved K3 8.84 mm to (68.1, 74.7)
- moved K1 7.17 mm to (68.1, 59.6), turned to 90 degrees
- moved Q1 6.41 mm to (91.4, 66.0)
- moved K5 6.22 mm to (68.1, 66.7), turned to 90 degrees
- moved R2 4.77 mm to (82.3, 64.9), turned to 90 degrees
- moved K4 4.44 mm to (68.1, 63.1), turned to 90 degrees
- moved Q2 4.33 mm to (86.4, 66.0)
- renumbered P1 to XBEE1
Connections:
- Q1 pad 1: GND -> /Sensor Block/USART To OneWire/nUSART_TX
- Q1 pad 3: Net-(Q1-Pad3) -> GND
- Q2 pad 1: Net-(Q2-Pad1) -> /Sensor Block/USART To OneWire/ONEWIRE_BUS
- Q2 pad 2: Net-(Q1-Pad3) -> /Sensor Block/USART To OneWire/nUSART_TX
- Q2 pad 3: /Sensor Block/USART To OneWire/ONEWIRE_BUS -> GND
- R2 pad 2: Net-(Q1-Pad3) -> /Sensor Block/USART To OneWire/nUSART_TX
- U2 pad 16: (no net) -> /Sensor Block/LIGHT1_FREQ
- U2 pad 19: /Sensor Block/USART To OneWire/DATA_EN -> (no net)
- U2 pad 29: /Sensor Block/LIGHT1_FREQ -> (no net)
- U2 pad 42: /Sensor Block/LIGHT2_FREQ -> /Sensor Block/IMU_SCL
- U2 pad 43: /Sensor Block/LIGHT2_EN -> /Sensor Block/IMU_SDA
- U2 pad 45: /Sensor Block/LIGHT2_SEL2 -> (no net)
- U2 pad 46: /Sensor Block/LIGHT2_SEL3 -> (no net)
Routing:
- net +3V3: track 301.0 -> 226.3 mm, vias 11 -> 7
- net /Sensor Block/LIGHT2_SEL3: track 47.2 -> 0.00 mm
- net /Sensor Block/LIGHT2_FREQ: track 47.0 -> 0.00 mm
- net /Sensor Block/LIGHT2_SEL2: track 44.2 -> 0.00 mm
- net /Sensor Block/IMU_SCL: track 0.00 -> 43.6 mm, vias 0 -> 1
- net /Sensor Block/IMU_SDA: track 0.00 -> 42.2 mm
- net /Sensor Block/LIGHT2_EN: track 42.0 -> 0.00 mm, vias 1 -> 0
- net GND: track 73.2 -> 92.0 mm
- net /Sensor Block/USART To OneWire/DATA_EN: track 12.8 -> 0.00 mm
- net Net-(Q1-Pad3): track 11.0 -> 0.00 mm
- net /Sensor Block/USART To OneWire/nUSART_TX: track 0.00 -> 10.2 mm
- net /Sensor Block/NOISE_LEVEL: track 20.8 -> 30.5 mm
- net Net-(Q2-Pad1): track 8.51 -> 0.00 mm
- net /Sensor Block/USART To OneWire/USART_TX: track 17.3 -> 8.97 mm, vias 1 -> 0
- net Net-(Q4-Pad3): track 6.90 -> 0.00 mm
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