File: sensor-node-ext/fab.kicad_pcb (KiCad board)
At the start: 2 copper layers, 199.5 x 150.8 mm, 170 parts, among them IC2 ENC28J60-I/SP, J1 DB9, J1 INSELECT, J2 RJ45-TRANSFO, J3 DB9, K1 XLR3, K2 XLR3, K3 XLR3, K4 XLR3, K5 XLR3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

Commit message: Clean up sensor-node-ext data
Parts:
- moved P2 271.7 mm to (270.7, 78.6), turned to 90 degrees
- moved R1 262.8 mm to (278.8, 49.9), turned to 180 degrees
- moved C11 261.4 mm to (262.8, 77.3), turned to 270 degrees
- moved IC2 258.1 mm to (262.8, 73.0), turned to 180 degrees
- moved P1 257.5 mm to (271.2, 57.2), turned to 270 degrees
- moved C3 250.7 mm to (257.5, 71.7), turned to 90 degrees
- moved C4 245.1 mm to (257.5, 64.1), turned to 90 degrees
- moved R6 245.0 mm to (268.7, 41.5), turned to 90 degrees
- moved R7 244.3 mm to (272.0, 31.3), turned to 270 degrees
- moved R2 240.2 mm to (265.6, 40.0), turned to 270 degrees
- moved C5 238.1 mm to (257.5, 53.9), turned to 270 degrees
- moved C2 234.8 mm to (257.5, 48.8), turned to 90 degrees
- moved C1 231.8 mm to (257.5, 43.8), turned to 270 degrees
- moved Y1 229.8 mm to (245.8, 62.6), turned to 270 degrees
- moved C8 229.1 mm to (240.2, 69.9), turned to 90 degrees
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Other:
- board size 199.5 x 150.8 mm -> 272.7 x 159.6 mm
